File: KiCad/BlockyTypeV0.2.3.kicad_pcb (KiCad board)
At the start: 2 copper layers, 165.1 x 108.9 mm, 75 parts

Commit message: generated the gerber files for the pcb
Parts:
- moved LED2 4.06 mm to (-11.9, -25.5)
- moved S10 4.06 mm to (50.5, -42.1)
- moved D15 4.06 mm to (62.9, -67.3)
- moved D11 4.06 mm to (42.9, -59.3)
- moved D16 4.06 mm to (82.9, -26.3)
- moved MH6 4.06 mm to (85.5, -11.1)
- moved S18 4.06 mm to (90.5, -63.1)
- moved LED16 4.06 mm to (90.5, -22.1)
- moved MH8 4.06 mm to (103.5, -28.1)
- moved LED19 4.06 mm to (96.4, -0.39)
- moved JST1 4.06 mm to (111.9, -3.06)
- moved D4 4.06 mm to (1.81, -19.0)
- moved LED4 4.06 mm to (10.0, -16.1)
- moved D7 4.06 mm to (22.9, -31.3)
- moved MH4 4.06 mm to (40.5, -40.6)
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Routing:
- net P21: track 222.7 -> 244.5 mm
- net P19: track 160.4 -> 167.9 mm
- net P16: track 110.2 -> 116.2 mm
- net P20: track 250.4 -> 247.7 mm
- net P18: track 192.1 -> 189.9 mm
- net P15: track 123.9 -> 125.3 mm
- net BAT_P: track 33.2 -> 32.0 mm
- net VCC_LED: track 549.6 -> 550.6 mm
- net GND: track 678.5 -> 679.2 mm
- net P4: track 173.0 -> 172.2 mm
- net P5: track 168.8 -> 168.3 mm
